Commit message: Add second UR5e arm with Shadow Hand and left controllers

File: ros2_ws/src/quest_teleop_description/urdf/ur5e_shadow.urdf.xacro (robot description, xacro)
@@ -36,5 +36,5 @@
     safety_k_position="$(arg safety_k_position)"
     force_abs_paths="$(arg force_abs_paths)">
-    <origin xyz="0 0 0" rpy="0 0 0"/>
+    <origin xyz="0 -0.3 0" rpy="0 0 0"/>
   </xacro:ur_robot>
   <xacro:shadow_hand prefix="hand_" parent="$(arg tf_prefix)tool0">
@@ -47,3 +47,28 @@
     initial_positions="${xacro.load_yaml(initial_positions_file)}"/>
   <xacro:shadow_hand_ros2_control name="shadow_hand" prefix="hand_"/>
+  <xacro:arg name="left_hand" default="false"/>
+  <xacro:ur_robot
+    name="left_ur"
+    tf_prefix="left_"
+    parent="world"
+    joint_limits_parameters_file="$(arg joint_limit_params)"
+    kinematics_parameters_file="$(arg kinematics_params)"
+    physical_parameters_file="$(arg physical_params)"
+    visual_parameters_file="$(arg visual_params)"
+    safety_limits="$(arg safety_limits)"
+    safety_pos_margin="$(arg safety_pos_margin)"
+    safety_k_position="$(arg safety_k_position)"
+    force_abs_paths="$(arg force_abs_paths)">
+    <origin xyz="0 0.3 0" rpy="0 0 0"/>
+  </xacro:ur_robot>
+  <xacro:ur_ros2_control
+    name="left_ur_arm"
+    tf_prefix="left_"
+    initial_positions="${xacro.load_yaml(initial_positions_file)}"/>
+  <xacro:if value="$(arg left_hand)">
+    <xacro:shadow_hand prefix="left_hand_" parent="left_tool0">
+      <origin xyz="$(arg hand_mount_xyz)" rpy="$(arg hand_mount_rpy)"/>
+    </xacro:shadow_hand>
+    <xacro:shadow_hand_ros2_control name="left_shadow_hand" prefix="left_hand_"/>
+  </xacro:if>
 </robot>
